File: board/MouseTrap.kicad_pcb (KiCad board)
At the start: 2 copper layers, 63.2 x 53 mm, 18 parts, among them J1 Barrier LED, J2 Barrier Sensor, J3 Solenoid, J4 Solenoid, Q1 IRLB8721PBF

Commit message: Update footprints with models
Parts:
- A1: footprint Module:Adafruit_Feather -> SaintGimp:Adafruit_Feather
- J1, J3: footprint TerminalBlock_TE-Connectivity:TerminalBlock_TE_282834-2_1x02_P2.54mm_Horizontal -> SaintGimp:TerminalBlock_TE_282834-2_1x02_P2.54mm_Horizontal
- J2: footprint TerminalBlock_TE-Connectivity:TerminalBlock_TE_282834-3_1x03_P2.54mm_Horizontal -> SaintGimp:TerminalBlock_TE_282834-3_1x03_P2.54mm_Horizontal
Changed lines of the file:
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@@
 		)
 	)
-	(footprint "TerminalBlock_TE-Connectivity:TerminalBlock_TE_282834-3_1x03_P2.54mm_Horizontal"
+	(footprint "SaintGimp:TerminalBlock_TE_282834-3_1x03_P2.54mm_Horizontal"
 		(layer "F.Cu")
 		(at 162.56 111.76)
@@
 			)
 			(rotate
-				(xyz -0 -0 -0)
+				(xyz 0 0 0)
 			)
 		)
@@
 		)
 	)
-	(footprint "TerminalBlock_TE-Connectivity:TerminalBlock_TE_282834-2_1x02_P2.54mm_Horizontal"
+	(footprint "SaintGimp:TerminalBlock_TE_282834-2_1x02_P2.54mm_Horizontal"
 		(layer "F.Cu")
 		(at 167.64 71.12 180)
@@
 		)
 	)
-	(footprint "Module:Adafruit_Feather"
-		(placed yes)
+	(footprint "SaintGimp:Adafruit_Feather"
 		(layer "F.Cu")
 		(at 172.72 81.28 -90)
@@
 		(tags "Adafruit Feather")
 		(property "Reference" "A1"
-			(at 10.16 -7.62 90)
+			(at 10.16 -7.62 270)
 			(layer "F.SilkS")
 			(effects
@@
 			(at 10.16 45.72 90)
 			(layer "F.Fab")
-			(hide yes)
 			(effects
 				(font
@@
 		)
 		(fp_text user "${REFERENCE}"
-			(at 10.16 19.05 0)
+			(at 10.16 19.05 180)
 			(layer "F.Fab")
 			(effects
@@
 			)
 		)
+		(model "D:/SaintGimp/KiCad/modules/packages3d/SaintGimp.3dshapes/3403 Feather M0 Express.step"
+			(offset
+				(xyz -1.275 6.35 11)
+			)
+			(scale
+				(xyz 1 1 1)
+			)
+			(rotate
+				(xyz -0 -0 90)
+			)
+		)
+		(model "${KICAD9_3DMODEL_DIR}/Connector_PinHeader_2.54mm.3dshapes/PinHeader_1x12_P2.54mm_Vertical.step"
+			(offset
+				(xyz 20.3 -10.2 11)
+			)
+			(scale
+				(xyz 1 1 1)
+			)
+			(rotate
+				(xyz -0 -180 -0)
+			)
+		)
+		(model "${KICAD9_3DMODEL_DIR}/Connector_PinHeader_2.54mm.3dshapes/PinHeader_1x16_P2.54mm_Vertical.step"
+			(offset
+				(xyz 0 0 11)
+			)
+			(scale
+				(xyz 1 1 1)
+			)
+			(rotate
+				(xyz -0 -180 -0)
+			)
+		)
+		(model "${KICAD9_3DMODEL_DIR}/Connector_PinSocket_2.54mm.3dshapes/PinSocket_1x16_P2.54mm_Vertical.step"
+			(offset
+				(xyz 0 0 0)
+			)
+			(scale
+				(xyz 1 1 1)
+			)
+			(rotate
+				(xyz 0 0 0)
+			)
+		)
+		(model "${KICAD9_3DMODEL_DIR}/Connector_PinSocket_2.54mm.3dshapes/PinSocket_1x12_P2.54mm_Vertical.step"
+			(offset
+				(xyz 20.3 -10.2 0)
+			)
+			(scale
+				(xyz 1 1 1)
+			)
+			(rotate
+				(xyz -0 -0 -0)
+			)
+		)
 	)
 	(footprint "Resistor_THT:R_Axial_DIN0207_L6.3mm_D2.5mm_P7.62mm_Horizontal"
@@
 		(embedded_fonts no)
 	)
-	(footprint "TerminalBlock_TE-Connectivity:TerminalBlock_TE_282834-2_1x02_P2.54mm_Horizontal"
+	(footprint "SaintGimp:TerminalBlock_TE_282834-2_1x02_P2.54mm_Horizontal"
 		(layer "F.Cu")
 		(at 123.19 83.82 -90)
@@
 		(tags "THT Terminal Block TE 282834-2 pitch 2.54mm size 5.54x6.5mm drill 1.1mm pad 2.1mm")
 		(property "Reference" "J3"
-			(at 1.27 -4.37 90)
+			(at -3.175 0 0)
 			(layer "F.SilkS")
 			(effects
@@
 		)
 		(property "Value" "Solenoid"
-			(at 1.27 4.37 90)
+			(at 1.27 4.37 270)
 			(layer "F.Fab")
 			(effects
@@
 		)
 		(property "Datasheet" "~"
-			(at 0 0 90)
+			(at 0 0 270)
 			(layer "F.Fab")
 			(hide yes)
@@
 		)
 		(property "Description" "Generic screw terminal, single row, 01x02, script generated (kicad-library-utils/schlib/autogen/connector/)"
-			(at 0 0 90)
+			(at 0 0 270)
 			(layer "F.Fab")
 			(hide yes)
@@
 		)
 		(fp_text user "${REFERENCE}"
-			(at 1.27 2 90)
+			(at 1.27 2 270)
 			(layer "F.Fab")
 			(effects

Commit message: Board updates
Connections:
- J2 pad 1: GND -> Net-(A1-D10)
- J2 pad 2: +3.3V -> GND
- J2 pad 3: Net-(A1-D10) -> +3.3V
Routing:
- net Net-(A1-D10): track 25.9 -> 19.4 mm
- net +3.3V: track 32.6 -> 31.5 mm
Other:
- board text added: "SaintGimp Mouse Trap v1.1"
- board text removed: "SaintGimp Mouse Trap v1.0"
Changed lines of the file:
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@@
 			(remove_unused_layers no)
 			(roundrect_rratio 0.119048)
-			(net 3 "GND")
+			(net 21 "Net-(A1-D10)")
 			(pinfunction "Pin_1")
 			(pintype "passive")
@@
 			(layers "*.Cu" "*.Mask")
 			(remove_unused_layers no)
-			(net 31 "+3.3V")
+			(net 3 "GND")
 			(pinfunction "Pin_2")
 			(pintype "passive")
@@
 			(layers "*.Cu" "*.Mask")
 			(remove_unused_layers no)
-			(net 21 "Net-(A1-D10)")
+			(net 31 "+3.3V")
 			(pinfunction "Pin_3")
 			(pintype "passive")
@@
 	)
 	(gr_text "3V3"
-		(at 163.83 117.475 0)
+		(at 167.64 117.475 0)
 		(layer "F.SilkS")
 		(effects
@@
 	)
 	(gr_text "OUT"
-		(at 167.64 117.475 0)
+		(at 160.02 117.475 0)
 		(layer "F.SilkS")
 		(effects
@@
 		)
 	)
-	(gr_text "SaintGimp\nMouse Trap v1.0"
+	(gr_text "SaintGimp\nMouse Trap v1.1"
 		(at 167.005 92.71 0)
 		(layer "F.SilkS")
@@
 	)
 	(gr_text "GND"
-		(at 160.02 117.475 0)
+		(at 163.83 117.475 0)
 		(layer "F.SilkS")
 		(effects
@@
 	)
 	(segment
-		(start 153.035 105.41)
-		(end 151.13 105.41)
+		(start 155.9814 105.1814)
+		(end 162.56 111.76)
 		(width 0.2)
 		(layer "F.Cu")
@@
 	)
 	(segment
-		(start 166.001 113.399)
-		(end 161.024 113.399)
+		(start 150.9014 105.1814)
+		(end 155.9814 105.1814)
 		(width 0.2)
 		(layer "F.Cu")
@@
 	)
 	(segment
-		(start 167.64 111.76)
-		(end 166.001 113.399)
-		(width 0.2)
-		(layer "F.Cu")
-		(net 21)
-	)
-	(segment
-		(start 151.13 105.41)
-		(end 147.32 101.6)
-		(width 0.2)
-		(layer "F.Cu")
-		(net 21)
-	)
-	(segment
-		(start 161.024 113.399)
-		(end 153.035 105.41)
+		(start 147.32 101.6)
+		(end 150.9014 105.1814)
 		(width 0.2)
 		(layer "F.Cu")
@@
 	)
 	(segment
-		(start 170.18 106.68)
+		(start 167.64 111.76)
+		(end 167.64 89.2302)
+		(width 0.2)
+		(layer "F.Cu")
+		(net 31)
+	)
+	(segment
+		(start 170.18 86.6902)
 		(end 170.18 81.28)
 		(width 0.2)
@@
 	)
 	(segment
-		(start 165.1 111.76)
-		(end 170.18 106.68)
+		(start 167.64 89.2302)
+		(end 170.18 86.6902)
 		(width 0.2)
 		(layer "F.Cu")
