File: board/MouseTrap.kicad_sch (KiCad schematic)
At the start: 14 parts, among them J1 Barrier LED, J2 Barrier Sensor, J3 Solenoid, J4 Solenoid, Q1 IRLB8721PBF

Commit message: Update footprints with models
Parts:
- A1: footprint Module:Adafruit_Feather -> SaintGimp:Adafruit_Feather
- J1, J3: footprint TerminalBlock_TE-Connectivity:TerminalBlock_TE_282834-2_1x02_P2.54mm_Horizontal -> SaintGimp:TerminalBlock_TE_282834-2_1x02_P2.54mm_Horizontal
- J2: footprint TerminalBlock_TE-Connectivity:TerminalBlock_TE_282834-3_1x03_P2.54mm_Horizontal -> SaintGimp:TerminalBlock_TE_282834-3_1x03_P2.54mm_Horizontal
Changed lines of the file:
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@@
 			)
 		)
-		(property "Footprint" "TerminalBlock_TE-Connectivity:TerminalBlock_TE_282834-2_1x02_P2.54mm_Horizontal"
+		(property "Footprint" "SaintGimp:TerminalBlock_TE_282834-2_1x02_P2.54mm_Horizontal"
 			(at 54.61 95.25 0)
 			(effects
@@
 			)
 		)
-		(property "Footprint" "TerminalBlock_TE-Connectivity:TerminalBlock_TE_282834-3_1x03_P2.54mm_Horizontal"
+		(property "Footprint" "SaintGimp:TerminalBlock_TE_282834-3_1x03_P2.54mm_Horizontal"
 			(at 66.04 81.28 0)
 			(effects
@@
 			)
 		)
-		(property "Footprint" "Module:Adafruit_Feather"
+		(property "Footprint" "SaintGimp:Adafruit_Feather"
 			(at 118.11 121.92 0)
 			(effects
@@
 			)
 		)
-		(property "Footprint" "TerminalBlock_TE-Connectivity:TerminalBlock_TE_282834-2_1x02_P2.54mm_Horizontal"
+		(property "Footprint" "SaintGimp:TerminalBlock_TE_282834-2_1x02_P2.54mm_Horizontal"
 			(at 66.04 74.93 0)
 			(effects

Commit message: Board updates
Connections:
- net +3.3V: now also J2.3 (Pin_3); no longer J2.2 (Pin_2)
- net GND: now also J2.2 (Pin_2); no longer J2.1 (Pin_1)
- net at A1.22 (D10): now also J2.1 (Pin_1); no longer J2.3 (Pin_3)
Changed lines of the file:
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@@
 	(wire
 		(pts
-			(xy 85.09 74.93) (xy 85.09 78.74)
+			(xy 85.09 74.93) (xy 85.09 83.82)
 		)
 		(stroke
@@
 	(wire
 		(pts
-			(xy 85.09 78.74) (xy 71.12 78.74)
+			(xy 71.12 83.82) (xy 85.09 83.82)
 		)
 		(stroke
@@
 	(symbol
 		(lib_id "power:+3.3V")
-		(at 71.12 81.28 270)
+		(at 71.12 78.74 270)
 		(unit 1)
 		(exclude_from_sim no)
@@
 		(fields_autoplaced yes)
 		(property "Reference" "#PWR06"
-			(at 67.31 81.28 0)
+			(at 67.31 78.74 0)
 			(effects
 				(font
@@
 		)
 		(property "Value" "+3.3V"
-			(at 74.93 81.2799 90)
+			(at 74.93 78.7399 90)
 			(effects
 				(font
@@
 		)
 		(property "Footprint" ""
-			(at 71.12 81.28 0)
+			(at 71.12 78.74 0)
 			(effects
 				(font
@@
 		)
 		(property "Datasheet" ""
-			(at 71.12 81.28 0)
+			(at 71.12 78.74 0)
 			(effects
 				(font
@@
 		)
 		(property "Description" "Power symbol creates a global label with name \"+3.3V\""
-			(at 71.12 81.28 0)
+			(at 71.12 78.74 0)
 			(effects
 				(font
@@
 	(symbol
 		(lib_id "power:GND")
-		(at 71.12 83.82 90)
+		(at 71.12 81.28 90)
 		(unit 1)
 		(exclude_from_sim no)
@@
 		(fields_autoplaced yes)
 		(property "Reference" "#PWR07"
-			(at 77.47 83.82 0)
+			(at 77.47 81.28 0)
 			(effects
 				(font
@@
 		)
 		(property "Value" "GND"
-			(at 74.93 83.8199 90)
+			(at 74.93 81.2799 90)
 			(effects
 				(font
@@
 		)
 		(property "Footprint" ""
-			(at 71.12 83.82 0)
+			(at 71.12 81.28 0)
 			(effects
 				(font
@@
 		)
 		(property "Datasheet" ""
-			(at 71.12 83.82 0)
+			(at 71.12 81.28 0)
 			(effects
 				(font
@@
 		)
 		(property "Description" "Power symbol creates a global label with name \"GND\" , ground"
-			(at 71.12 83.82 0)
-			(effects
-				(font
+			(at 71.12 81.28 0)
+			(effects
+				(font
